Commit message: 0206備份

File: wheeltec_robot_urdf/wheeltec_robot_urdf/urdf/mini_mec_robot.urdf (robot description, URDF)
Before this commit: robot wheeltec_robot, 5 links, 4 joints
Joints:
- joint right_wheel_joint: origin xyz=--0.325 -0.3285 0.09 rpy=1.57 0 0 -> xyz=-0.325 -0.3285 0.09 rpy=1.57 0 0
